Commit message: Fixing the gripper

File: robotic_arm_environment/arm_pkg/urdf/manipulator.xacro (robot description, xacro)
@@ -3,4 +3,5 @@
     <xacro:include filename="$(find arm_pkg)/urdf/a0912.urdf.xacro" />
     <xacro:include filename="$(find arm_pkg)/urdf/depth_camera.xacro"/>
+    <xacro:include filename="$(find robotiq_85_description)/urdf/robotiq_85_gripper_macro_gz.urdf.xacro" />
     <xacro:manipulator namespace=""/>
     <link name="world">
@@ -26,12 +27,15 @@
         <child link="base_0"/>
     </joint>
-    <!-- Load Common Material -->
+    <xacro:robotiq_85_gripper prefix="" parent="link6" >
+       <origin xyz="0.0 0 0.0" rpy="0 -1.57 1.57"/>
+    </xacro:robotiq_85_gripper>
+    <!-- Load Common Material >
     <xacro:include filename="$(find xarm_description)/urdf/common/common.material.xacro" />
-    <xacro:common_material prefix=""/>
-    <!-- Specify Mesh file path -->
-    <xacro:property name="mesh_suffix" value="stl"/>
-    <!-- gazebo use -->
-    <xacro:property name="mesh_path" value="file://$(find xarm_description)/meshes" />
-    <!-- include the GRIPPER -->
+    <xacro:common_material prefix=""/-->
+    <!-- Specify Mesh file path >
+    <xacro:property name="mesh_suffix" value="stl"/-->
+    <!-- gazebo use >
+    <xacro:property name="mesh_path" value="file://$(find xarm_description)/meshes" /-->
+    <!-- include the GRIPPER >
     <xacro:include filename="$(find xarm_description)/urdf/common/common.link.xacro" />
     <xacro:parse_link_inertial_filename dof="6" robot_type="xarm" robot_sn="" model1300="false" />
@@ -39,4 +43,4 @@
     <xacro:property name="new_model1300" value="${scope_parent_model1300}"/>
     <xacro:include filename="$(find xarm_description)/urdf/gripper/xarm_gripper_macro.xacro" />
-    <xacro:xarm_gripper_macro prefix="" attach_to="link6" ros2_control_plugin="gazebo_ros2_control/GazeboSystem" dof="6" hard_interface="PositionJointInterface" />
+    <xacro:xarm_gripper_macro prefix="" attach_to="link6" ros2_control_plugin="gazebo_ros2_control/GazeboSystem" dof="6" hard_interface="PositionJointInterface" /-->
 </robot>
