Commit message: Fixing the gripper

File: moveit_config/config/robot_description.ros2_control.xacro (robot description, xacro)
@@ -9,51 +9,16 @@
             </hardware>
             <joint name="joint1">
-                <command_interface name="position"/>
-                <state_interface name="position">
-                  <param name="initial_value">${initial_positions['joint1']}</param>
-                </state_interface>
-                <state_interface name="velocity"/>
             </joint>
             <joint name="joint2">
-                <command_interface name="position"/>
-                <state_interface name="position">
-                  <param name="initial_value">${initial_positions['joint2']}</param>
-                </state_interface>
-                <state_interface name="velocity"/>
             </joint>
             <joint name="joint3">
-                <command_interface name="position"/>
-                <state_interface name="position">
-                  <param name="initial_value">${initial_positions['joint3']}</param>
-                </state_interface>
-                <state_interface name="velocity"/>
             </joint>
             <joint name="joint4">
-                <command_interface name="position"/>
-                <state_interface name="position">
-                  <param name="initial_value">${initial_positions['joint4']}</param>
-                </state_interface>
-                <state_interface name="velocity"/>
             </joint>
             <joint name="joint5">
-                <command_interface name="position"/>
-                <state_interface name="position">
-                  <param name="initial_value">${initial_positions['joint5']}</param>
-                </state_interface>
-                <state_interface name="velocity"/>
             </joint>
             <joint name="joint6">
-                <command_interface name="position"/>
-                <state_interface name="position">
-                  <param name="initial_value">${initial_positions['joint6']}</param>
-                </state_interface>
-                <state_interface name="velocity"/>
             </joint>
-            <joint name="drive_joint">
-                <command_interface name="position"/>
-                <state_interface name="position">
-                  <param name="initial_value">${initial_positions['drive_joint']}</param>
-                </state_interface>
-                <state_interface name="velocity"/>
+            <joint name="robotiq_85_left_knuckle_joint">
             </joint>
         </ros2_control>

File: robotic_arm_environment/arm_pkg/urdf/manipulator.xacro (robot description, xacro)
@@ -30,17 +30,3 @@
        <origin xyz="0.0 0 0.0" rpy="0 -1.57 1.57"/>
     </xacro:robotiq_85_gripper>
-    <!-- Load Common Material >
-    <xacro:include filename="$(find xarm_description)/urdf/common/common.material.xacro" />
-    <xacro:common_material prefix=""/-->
-    <!-- Specify Mesh file path >
-    <xacro:property name="mesh_suffix" value="stl"/-->
-    <!-- gazebo use >
-    <xacro:property name="mesh_path" value="file://$(find xarm_description)/meshes" /-->
-    <!-- include the GRIPPER >
-    <xacro:include filename="$(find xarm_description)/urdf/common/common.link.xacro" />
-    <xacro:parse_link_inertial_filename dof="6" robot_type="xarm" robot_sn="" model1300="false" />
-    <xacro:property name="inertial_params_filename" value="${scope_parent_inertial_params_filename}"/>
-    <xacro:property name="new_model1300" value="${scope_parent_model1300}"/>
-    <xacro:include filename="$(find xarm_description)/urdf/gripper/xarm_gripper_macro.xacro" />
-    <xacro:xarm_gripper_macro prefix="" attach_to="link6" ros2_control_plugin="gazebo_ros2_control/GazeboSystem" dof="6" hard_interface="PositionJointInterface" /-->
 </robot>
